File: final_kicad/final.kicad_pcb (KiCad board)
At the start: 2 copper layers, 12 parts, among them M1 Motor_DC, Q1 NPN, SW1 SW_Push, SW3 SW_SPST, U1 XIAO-ESP32-C3-SMD, U2 MPU-6050

Commit message: line
Parts:
- moved D1 68.7 mm to (93.0, 38.5), turned to 90 degrees
- moved R1 68.0 mm to (72.8, 55.0)
- moved FSR400 62.7 mm to (67.5, 74.0), turned to 90 degrees
- moved R2 59.6 mm to (72.0, 98.8)
- moved Q1 47.1 mm to (102.5, 41.0), turned to 180 degrees
- moved U2 42.0 mm to (84.8, 84.2)
- moved SW1 40.3 mm to (78.0, 81.5), turned to 180 degrees
- moved SW3 29.3 mm to (118.5, 60.5)
- moved BT1 20.8 mm to (127.8, 50.3), turned to 180 degrees
- moved M1 18.2 mm to (141.0, 69.8), turned to -90 degrees
- moved U1 13.9 mm to (99.0, 72.0)
- moved C1 0.57 mm to (143.5, 83.5), turned to -90 degrees
Routing:
- net Net-(BT1-+): track 0.00 -> 185.9 mm
- net GND: track 0.00 -> 78.0 mm
- net Net-(U1-GPIO3_A1_D1): track 0.00 -> 77.6 mm
- net Net-(M1--): track 0.00 -> 55.8 mm
- net Net-(U1-GPIO5_A3_D3): track 0.00 -> 37.6 mm
- net Net-(SW3-B): track 0.00 -> 37.2 mm
- net Net-(D1-A): track 0.00 -> 28.1 mm
- net Net-(Q1-B): track 0.00 -> 27.1 mm
- net Net-(U1-GPIO4_A2_D2): track 0.00 -> 23.4 mm
- net Net-(SW3-A): track 0.00 -> 22.2 mm
- net Net-(BT1--): track 0.00 -> 18.0 mm
- net Net-(U1-GPIO6_D4_SDA): track 0.00 -> 11.6 mm
- net Net-(U1-GPIO7_D5_SCL): track 0.00 -> 9.47 mm
