File: final_kicad/_autosave-final.kicad_pcb (KiCad board)
At the start: 2 copper layers, 10 x 95.5 mm, 19 parts, among them J1 Signal, J2 Battery, J3 Power, M1 Motor_DC, Q1 NPN, SW1 SW_SPST, SW2 SW_Push, U1 MPU-6050

Commit message: 1
Routing:
- net Net-(D1-K): track 175.4 -> 183.2 mm, vias 0 -> 2
Changed lines of the file:
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@@
-	)
-	(segment
-		(start 157.7 78.7)
-		(end 157.7 77.2)
-		(width 0.2)
-		(layer "F.Cu")
-		(net 2)
 	)
 	(segment
@@
 	)
 	(segment
+		(start 153.8 78.7)
+		(end 152.1 77)
+		(width 0.2)
+		(layer "F.Cu")
+		(net 2)
+	)
+	(segment
 		(start 156.2 57.5)
 		(end 156 57.7)
@@
 	)
 	(segment
+		(start 157.7 78)
+		(end 157.7 77.2)
+		(width 0.2)
+		(layer "F.Cu")
+		(net 2)
+	)
+	(segment
 		(start 159.25 108.75)
 		(end 159.25 44.3)
@@
 	)
 	(segment
+		(start 152.1 77)
+		(end 152 77)
+		(width 0.2)
+		(layer "F.Cu")
+		(net 2)
+	)
+	(segment
 		(start 159.275 29.825)
 		(end 159.275 39.675)
@@
 	)
 	(segment
+		(start 157.7 78.7)
+		(end 157.7 78)
+		(width 0.2)
+		(layer "F.Cu")
+		(net 2)
+	)
+	(segment
 		(start 157.5 62)
 		(end 156.2 60.7)
@@
 		(net 2)
 	)
+	(via
+		(at 152 77)
+		(size 0.6)
+		(drill 0.3)
+		(layers "F.Cu" "B.Cu")
+		(net 2)
+	)
+	(via
+		(at 157.1 76.5)
+		(size 0.6)
+		(drill 0.3)
+		(layers "F.Cu" "B.Cu")
+		(net 2)
+	)
+	(segment
+		(start 156.6 77)
+		(end 157.1 76.5)
+		(width 0.2)
+		(layer "B.Cu")
+		(net 2)
+	)
+	(segment
+		(start 152 77)
+		(end 156.6 77)
+		(width 0.2)
+		(layer "B.Cu")
+		(net 2)
+	)
