File: final_kicad/_autosave-final.kicad_sch (KiCad schematic)
At the start: 19 parts, among them J1 Signal, J2 Battery, J3 Power, M1 Motor_DC, Q1 NPN, SW1 SW_SPST, SW2 SW_Push, U1 MPU-6050

Commit message: 1
Parts:
- added C6, C7, C9: 0.1U, Capacitor_SMD:C_0603_1608Metric, symbol Device:C
- added C8: 2200PF, Capacitor_SMD:C_0603_1608Metric, symbol Device:C
- added D2: LED, LED_THT:LED_D3.0mm, symbol Device:LED
- added FSR1: 10K, Connector_PinHeader_1.00mm:PinHeader_1x02_P1.00mm_Vertical, symbol Device:R_Variable
- added J4: SDA, symbol Connector:Conn_01x01_Pin
- added J5: Signal, Connector_PinHeader_1.00mm:PinHeader_1x06_P1.00mm_Vertical, symbol Connector:Conn_01x06_Pin
- added J7: SCL, symbol Connector:Conn_01x01_Pin
- added M2: Motor_DC, Connector_PinHeader_1.00mm:PinHeader_1x02_P1.00mm_Vertical, symbol Motor:Motor_DC
- added Q2: NPN, Crystal:Resonator-3Pin_W6.0mm_H3.0mm, symbol Simulation_SPICE:NPN
- added R10: 10k, Resistor_SMD:R_0603_1608Metric, symbol Device:R
- added R5: 200, Resistor_SMD:R_0603_1608Metric, symbol Device:R
- added R6, R7: 4.7K, Resistor_SMD:R_0603_1608Metric, symbol Device:R
- added SW3: SW_Push, Button_Switch_THT:SW_PUSH_6mm, symbol Switch:SW_Push
- added U2: MPU-6050, Sensor_Motion:InvenSense_QFN-24_4x4mm_P0.5mm, symbol Sensor_Motion:MPU-6050
Connections:
- new net: C8.1, U2.20 (CPOUT)
- new net: J4.1 (Pin_1), R6.2, U2.24 (SDA)
- new net: FSR1.1, J5.5 (Pin_5)
- new net: D2.2 (A), R5.2
- new net: J5.4 (Pin_4), R10.1, SW3.1
- new net: J5.6 (Pin_6), R5.1
- new net: C6.2, U2.10 (REGOUT)
- new net: J7.1 (Pin_1), R7.2, U2.23 (SCL)
- new net: J5.3 (Pin_3), Q2.2 (B)
- new net +3V3: C7.1, C9.2, R10.2, R6.1, R7.1, U2.13 (VDD), U2.8 (VLOGIC)
- new net GND: C6.1, C7.2, C8.2, C9.1, D2.1 (K), FSR1.2, M2.1 (+), Q2.3 (E), SW3.2, U2.1 (CLKIN), U2.18 (GND)
- no-connect marks 4 -> 15
